File: driving-control-device.kicad_sch (KiCad schematic)
At the start: 6 parts, among them J1 Micro_SD_Card, U1 MPU-6050, U2 NEO-M9N, U3 SIM7020C

Commit message: upd: principial schematic
Connections:
- net at U3.1 (UART1_TXD): now also A1.10 (TX), A2.16 (D1/TX), U2.20 (TXD/SPI_MISO)
- net at U3.2 (UART1_RXD): now also A1.11 (RX), A2.15 (D0/RX), U2.21 (RXD/SPI_MOSI)
- now unconnected: U3.22 (UART2_TXD), U3.23 (UART2_RXD)
- no-connect marks 26 -> 63
Changed lines of the file:
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@@
+	)
+	(no_connect
+		(at 311.15 111.76)
+	)
+	(no_connect
+		(at 81.28 91.44)
+	)
+	(no_connect
+		(at 311.15 119.38)
+	)
+	(no_connect
+		(at 96.52 43.18)
 	)
 	(no_connect
@@
 	)
 	(no_connect
+		(at 339.09 92.71)
+	)
+	(no_connect
+		(at 81.28 55.88)
+	)
+	(no_connect
+		(at 121.92 60.96)
+	)
+	(no_connect
+		(at 81.28 88.9)
+	)
+	(no_connect
+		(at 121.92 68.58)
+	)
+	(no_connect
 		(at 123.19 128.27)
 	)
@@
 	)
 	(no_connect
+		(at 339.09 119.38)
+	)
+	(no_connect
+		(at 311.15 104.14)
+	)
+	(no_connect
+		(at 311.15 100.33)
+	)
+	(no_connect
+		(at 339.09 96.52)
+	)
+	(no_connect
+		(at 121.92 48.26)
+	)
+	(no_connect
 		(at 143.51 143.51)
 	)
@@
 	)
 	(no_connect
+		(at 311.15 107.95)
+	)
+	(no_connect
+		(at 121.92 86.36)
+	)
+	(no_connect
+		(at 81.28 83.82)
+	)
+	(no_connect
+		(at 339.09 100.33)
+	)
+	(no_connect
+		(at 81.28 50.8)
+	)
+	(no_connect
 		(at 143.51 153.67)
 	)
 	(no_connect
+		(at 121.92 83.82)
+	)
+	(no_connect
 		(at 256.54 52.07)
 	)
@@
 	)
 	(no_connect
+		(at 339.09 107.95)
+	)
+	(no_connect
+		(at 106.68 43.18)
+	)
+	(no_connect
 		(at 233.68 142.24)
 	)
@@
 	)
 	(no_connect
+		(at 81.28 53.34)
+	)
+	(no_connect
 		(at 276.86 74.93)
 	)
 	(no_connect
+		(at 121.92 63.5)
+	)
+	(no_connect
+		(at 121.92 76.2)
+	)
+	(no_connect
 		(at 241.3 77.47)
 	)
 	(no_connect
+		(at 339.09 104.14)
+	)
+	(no_connect
 		(at 241.3 59.69)
 	)
 	(no_connect
+		(at 81.28 48.26)
+	)
+	(no_connect
 		(at 241.3 82.55)
 	)
 	(no_connect
+		(at 121.92 91.44)
+	)
+	(no_connect
+		(at 121.92 58.42)
+	)
+	(no_connect
 		(at 241.3 87.63)
 	)
 	(no_connect
+		(at 121.92 66.04)
+	)
+	(no_connect
+		(at 121.92 78.74)
+	)
+	(no_connect
+		(at 311.15 115.57)
+	)
+	(no_connect
+		(at 81.28 68.58)
+	)
+	(no_connect
 		(at 241.3 90.17)
 	)
 	(no_connect
+		(at 121.92 73.66)
+	)
+	(no_connect
+		(at 81.28 58.42)
+	)
+	(no_connect
 		(at 241.3 62.23)
 	)
 	(no_connect
+		(at 121.92 93.98)
+	)
+	(no_connect
+		(at 81.28 71.12)
+	)
+	(no_connect
 		(at 107.95 143.51)
 	)
@@
 	(wire
 		(pts
-			(xy 81.28 71.12) (xy 77.47 71.12)
-		)
-		(stroke
-			(width 0)
-			(type default)
-		)
-	)
-	(wire
-		(pts
 			(xy 254 48.26) (xy 254 52.07)
 		)
@@
 	(wire
 		(pts
-			(xy 77.47 71.12) (xy 77.47 116.84)
+			(xy 77.47 63.5) (xy 77.47 116.84)
 		)
 		(stroke
@@
 	(wire
 		(pts
-			(xy 73.66 68.58) (xy 73.66 119.38)
-		)
-		(stroke
-			(width 0)
-			(type default)
-		)
-	)
-	(wire
-		(pts
 			(xy 311.15 96.52) (xy 300.99 96.52)
 		)
@@
 	(wire
 		(pts
+			(xy 73.66 60.96) (xy 73.66 119.38)
+		)
+		(stroke
+			(width 0)
+			(type default)
+		)
+	)
+	(wire
+		(pts
 			(xy 104.14 140.97) (xy 107.95 140.97)
 		)
@@
 	(wire
 		(pts
+			(xy 77.47 63.5) (xy 81.28 63.5)
+		)
+		(stroke
+			(width 0)
+			(type default)
+		)
+	)
+	(wire
+		(pts
 			(xy 241.3 69.85) (xy 156.21 69.85)
 		)
@@
 	(wire
 		(pts
-			(xy 81.28 68.58) (xy 73.66 68.58)
-		)
-		(stroke
-			(width 0)
-			(type default)
-		)
-	)
-	(wire
-		(pts
 			(xy 161.29 92.71) (xy 161.29 144.78)
 		)
@@
 		)
 		(stroke
+			(width 0)
+			(type default)
+		)
+	)
+	(wire
+		(pts
+			(xy 73.66 60.96) (xy 81.28 60.96)
+		)
+		(stroke
